File: blueprint/design/pcb/goalfinder-tof-module/goalfinder-tof-module.kicad_sch (KiCad schematic)
At the start: 1 part, among them U1 VL53L8CXV0GC/1

Commit message: progress: #144
Parts:
- added U2: SN74AVC8T245RHLR, symbol SN74AVC8T245RHLR:SN74AVC8T245RHLR
- added U3: VL53L8CXV0GC/1, symbol VL53L8CXV0GC:VL53L8CXV0GC/1
- U1: footprint Library:VL53L5CXV0GC-1 -> (none)
Connections:
- net GND: now also U1.A7 (RSVD2)
